File: Digitales_MEGA/DigitalesSCH.sch (EAGLE design)
At the start: 26 parts

Commit message: Actaulización PCB y SCH
Connections:
- net 3V3: now also U$2.VCC
- net 5VDC: no longer U$2.VCC
Changed lines of the file:
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@@
 <label x="1460.5" y="1432.56" size="1.778" layer="95" xref="yes"/>
+</segment>
+<segment>
+<pinref part="U$2" gate="G$1" pin="VCC"/>
+<wire x1="1717.04" y1="1432.56" x2="1722.12" y2="1432.56" width="0.1524" layer="91"/>
+<label x="1722.12" y="1432.56" size="1.778" layer="95" xref="yes"/>
 </segment>
 </net>
@@
 <label x="1605.28" y="1389.38" size="1.778" layer="95" rot="R180" xref="yes"/>
 </segment>
-<segment>
-<pinref part="U$2" gate="G$1" pin="VCC"/>
-<wire x1="1717.04" y1="1432.56" x2="1722.12" y2="1432.56" width="0.1524" layer="91"/>
-<label x="1722.12" y="1432.56" size="1.778" layer="95" xref="yes"/>
-</segment>
 </net>
