File: Digitales_MEGA/DigitalesSCH.sch (EAGLE design)
At the start: 23 parts

Commit message: z
Parts:
- added S2: (no value), switch:M9040P
- added VIN, VOUT: 1X2-3.5MM, adafruit:1X2-3.5MM
Connections:
- new net N$14: S2.S, VOUT.1
- new net N$15: VIN.1, VOUT.2
- new net N$5: S2.P, VIN.2
- net 3V3: now also U$2.VCC
- net 5VDC: no longer U$2.VCC
Changed lines of the file:
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@@
 <part name="D_AUX2" library="adafruit" deviceset="PINHD-1X6" device=""/>
 <part name="D_AUX1" library="pinhead" library_urn="urn:adsk.eagle:library:325" deviceset="PINHD-1X5" device="" package3d_urn="urn:adsk.eagle:package:22469/2"/>
+<part name="VIN" library="adafruit" deviceset="1X2" device="-3.5MM"/>
+<part name="VOUT" library="adafruit" deviceset="1X2" device="-3.5MM"/>
+<part name="S2" library="switch" library_urn="urn:adsk.eagle:library:380" deviceset="M9040P" device="" package3d_urn="urn:adsk.eagle:package:27676/1"/>
 </parts>
 <sheets>
@@
 <instance part="D_AUX1" gate="A" x="1595.12" y="1430.02" smashed="yes">
 <attribute name="VALUE" x="1588.77" y="1419.86" size="1.778" layer="96"/>
+</instance>
+<instance part="VIN" gate="G$1" x="1457.96" y="1463.04" smashed="yes" rot="R180"/>
+<instance part="VOUT" gate="G$1" x="1488.44" y="1457.96" smashed="yes"/>
+<instance part="S2" gate="1" x="1470.66" y="1465.58" smashed="yes" rot="R270">
+<attribute name="NAME" x="1468.755" y="1471.93" size="1.778" layer="95"/>
+<attribute name="VALUE" x="1473.2" y="1469.39" size="1.778" layer="96"/>
 </instance>
 </instances>
@@
 <label x="1460.5" y="1432.56" size="1.778" layer="95" xref="yes"/>
 </segment>
+<segment>
+<pinref part="U$2" gate="G$1" pin="VCC"/>
+<wire x1="1717.04" y1="1432.56" x2="1722.12" y2="1432.56" width="0.1524" layer="91"/>
+<label x="1722.12" y="1432.56" size="1.778" layer="95" xref="yes"/>
+</segment>
 </net>
 <net name="5VDC" class="0">
@@
 <wire x1="1612.9" y1="1389.38" x2="1605.28" y2="1389.38" width="0.1524" layer="91"/>
 <label x="1605.28" y="1389.38" size="1.778" layer="95" rot="R180" xref="yes"/>
-</segment>
-<segment>
-<pinref part="U$2" gate="G$1" pin="VCC"/>
-<wire x1="1717.04" y1="1432.56" x2="1722.12" y2="1432.56" width="0.1524" layer="91"/>
-<label x="1722.12" y="1432.56" size="1.778" layer="95" xref="yes"/>
 </segment>
 </net>
@@
 </segment>
 </net>
+<net name="N$5" class="0">
+<segment>
+<pinref part="VIN" gate="G$1" pin="2"/>
+<wire x1="1463.04" y1="1463.04" x2="1465.58" y2="1463.04" width="0.1524" layer="91"/>
+<pinref part="S2" gate="1" pin="P"/>
+</segment>
+</net>
+<net name="N$14" class="0">
+<segment>
+<wire x1="1475.74" y1="1460.5" x2="1483.36" y2="1460.5" width="0.1524" layer="91"/>
+<pinref part="VOUT" gate="G$1" pin="1"/>
+<pinref part="S2" gate="1" pin="S"/>
+</segment>
+</net>
+<net name="N$15" class="0">
+<segment>
+<pinref part="VIN" gate="G$1" pin="1"/>
+<wire x1="1463.04" y1="1460.5" x2="1468.12" y2="1460.5" width="0.1524" layer="91"/>
+<wire x1="1468.12" y1="1460.5" x2="1468.12" y2="1457.96" width="0.1524" layer="91"/>
+<pinref part="VOUT" gate="G$1" pin="2"/>
+<wire x1="1468.12" y1="1457.96" x2="1483.36" y2="1457.96" width="0.1524" layer="91"/>
+</segment>
+</net>
