File: Digitales_MEGA/DigitalesSCH.brd (EAGLE design)
At the start: 92.5 x 59.6 mm, 23 parts

Commit message: z
Parts:
- added S2: (no value), switch:M9040P
- added VIN, VOUT: 1X2-3.5MM, adafruit:1X2-3.5MM
- moved LED1 1.27 mm to (19.1, 33.0)
- moved LED2 1.27 mm to (19.1, 38.1)
- moved LED3 1.27 mm to (19.1, 43.2)
- moved R1 1.27 mm to (25.4, 33.0)
- moved R2 1.27 mm to (25.4, 38.1)
- moved R3 1.27 mm to (25.4, 43.2)
- moved LED4 1.27 mm to (19.1, 48.3)
- moved R4 1.27 mm to (25.4, 48.3)
Connections:
- new net N$14: S2.3, VOUT.1
- new net N$15: VIN.1, VOUT.2
- new net N$5: S2.2, VIN.2
- net 3V3: now also U$2.VCC
- net 5VDC: no longer U$2.VCC
Routing:
- net N$5: track 0.00 -> 25.0 mm
- net 3V3: track 126.9 -> 144.0 mm, vias 0 -> 2
- net N$14: track 0.00 -> 8.52 mm
- net N$15: track 0.00 -> 4.12 mm
- net 5VDC: track 150.2 -> 146.9 mm
- net D11: track 22.9 -> 21.6 mm
- net D13: track 10.6 -> 9.36 mm
- net D12: track 17.4 -> 16.8 mm
- net D10: track 29.7 -> 29.2 mm
- added copper zone on layer 16, net AA0
- added copper zone on layer 16, net AA1
- removed copper zone on layer 16, net A
